File: jieliDFUtrigger.kicad_pcb (KiCad board)
At the start: 2 copper layers, 24.4 x 30 mm, 29 parts, among them J1 USB_C_Receptacle_USB2.0_16P, J2 USB_C_Receptacle_USB2.0_16P, J3 Conn_01x06, SW1 SW_Push, SW2 SW_DPDT_x2, U1 ATtiny412-SSNR

Commit message: Minor oversights
Parts:
- added C1: 1u, Capacitor_SMD:C_0402_1005Metric, F.Cu at (88.1, 33.8)
- turned JP2 to 0 degrees
Routing:
- net GND: vias 9 -> 8
